File: PCB/WMS/WMS/DataAcquisition.kicad_sch (KiCad schematic)
At the start: 2 parts

Commit message: +Update PCB (v.1)
membuat PCB versi 1
Parts:
- removed U5: ~, WMS_components:GM67_Barcode_Scanner, symbol WMS_components:GM67_Barcode_Scanner
- added U7: ~, WMS_components:YR903_RFID_Scanner_FPC, symbol WMS_components:YR903_RFID_module
Connections:
- net GND_DATA_ACQ: now also U7.12 (GND), U7.13 (GND), U7.3 (GND), U7.4 (GND), U7.8 (GND), U7.9 (GND)
- net POWER_RFID: now also U7.1 (VCC), U7.2 (VCC)
- net RX_RFID: now also U7.16 (RXD)
- net TX_RFID: now also U7.17 (TXD)
