File: PCB/WMS/WMS/Display.kicad_sch (KiCad schematic)
At the start: 6 parts

Commit message: +Update PCB (v.1)
membuat PCB versi 1
Parts:
- Brd1: footprint WMS_components:128x64OLED -> WMS_components:128x64OLED_v2
Changed lines of the file:
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@@
   (title_block
     (title "Subsistem Display")
-    (date "2024-02-28")
-    (rev "1.4")
+    (date "2024-03-05")
+    (rev "1.5")
     (company "Institut Teknologi Bandung")
     (comment 1 "Bostang Palaguna")
@@
       (effects (font (size 1.27 1.27)) hide)
     )
-    (pin "2")
-    (pin "1")
+    (pin "1")
+    (pin "2")
     (instances
       (project "WMS"
@@
       (effects (font (size 1.27 1.27)) (justify right) hide)
     )
-    (property "Footprint" "WMS_components:128x64OLED" (at 67.31 33.02 0)
+    (property "Footprint" "WMS_components:128x64OLED_v2" (at 67.31 33.02 0)
       (effects (font (size 1.27 1.27)) hide)
     )
@@
       (effects (font (size 1.27 1.27)) hide)
     )
+    (pin "1")
+    (pin "2")
+    (pin "3")
     (pin "4")
-    (pin "3")
-    (pin "2")
-    (pin "1")
     (instances
       (project "WMS"
@@
       (effects (font (size 1.27 1.27)) hide)
     )
-    (pin "2")
-    (pin "1")
+    (pin "1")
+    (pin "2")
     (instances
       (project "WMS"
@@
       (effects (font (size 1.27 1.27)) hide)
     )
-    (pin "2")
-    (pin "1")
+    (pin "1")
+    (pin "2")
     (instances
       (project "WMS"
@@
       (effects (font (size 1.27 1.27)) hide)
     )
-    (pin "2")
-    (pin "1")
-    (instances
-      (project "WMS"
+    (pin "1")
+    (pin "2")
+    (instances
+      (project "WMS"
