File: PCB/WMS/WMS/PSoC.kicad_sch (KiCad schematic)
At the start: 9 parts, among them J1 Conn_01x40_Socket, J2 Conn_01x40_Socket, J3 Conn_01x03_Socket, SW1 SW_Push_Open, SW3 SW_Push_Open, SW4 SW_SPDT

Commit message: +Update PCB (v.1)
membuat PCB versi 1
Parts:
- added U5: ~, WMS_components:Quad_SPI_flash_microSD_v2, symbol WMS_components:QUAD_SPI_and_MICRO_SD
- U6: footprint WMS_components:CY8CPROTO-062-4343W -> WMS_components:CY8CPROTO-062-4343W_v2
Connections:
- net GND: now also U5.1 (GND)
- net P11_2: now also U5.16 (11_2)
- net P11_3: now also U5.17 (11_3)
- net P11_4: now also U5.18 (11_4)
- net P11_5: now also U5.14 (11_5)
- net P11_6: now also U5.13 (11_6)
- net P11_7: now also U5.15 (11_7)
- net P12_0: now also U5.11 (12_0)
- net P12_1: now also U5.10 (12_1)
- net P12_4: now also U5.9 (12_4)
- net P12_5: now also U5.12 (12_5)
- net P13_0: now also U5.4 (13_0)
- net P13_1: now also U5.7 (13_1)
- net P13_2: now also U5.6 (13_2)
- net P13_3: now also U5.5 (13_3)
- net P13_4: now also U5.3 (13_4)
- net P13_5: now also U5.2 (13_5)
- net VDDIO_0: now also U5.8 (VDDIO_0)
Other:
- note added: "Connections & Hierarchical Pins"
- note added: "Quad SPI Flash & microSD Card"
- note removed: "Connections"
- note removed: "Hierarchical Pins"
- moved on the sheet: J1, J2, J3
