File: PCB/WMS/WMS/Power.kicad_sch (KiCad schematic)
At the start: 4 parts

Commit message: +Update PCB (v.1)
membuat PCB versi 1
Parts:
- U1: footprint WMS_components:YX850 -> WMS_components:YX850_v2
- U2: footprint WMS_components:MT3608_module -> WMS_components:MT3608_module_v2
- U3: footprint WMS_components:TP4056-18650 -> WMS_components:TP4056-18650_v2
Changed lines of the file:
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@@
   (title_block
     (title "Subsistem Power")
-    (date "2024-02-28")
-    (rev "1.4")
+    (date "2024-03-05")
+    (rev "1.5")
     (company "Institut Teknologi Bandung")
     (comment 1 "Bostang Palaguna")
@@
       (effects (font (size 1.27 1.27)) hide)
     )
+    (pin "1")
     (pin "2")
-    (pin "1")
     (instances
       (project "WMS"
@@
       (effects (font (size 1.27 1.27)))
     )
-    (property "Footprint" "WMS_components:YX850" (at 106.68 41.91 0)
+    (property "Footprint" "WMS_components:YX850_v2" (at 106.68 41.91 0)
       (effects (font (size 1.27 1.27)) hide)
     )
@@
     )
     (pin "1")
+    (pin "2")
     (pin "3")
-    (pin "6")
     (pin "4")
     (pin "5")
-    (pin "2")
+    (pin "6")
     (instances
       (project "WMS"
@@
       (effects (font (size 1.27 1.27)) hide)
     )
-    (property "Footprint" "WMS_components:TP4056-18650" (at 36.83 25.4 0)
+    (property "Footprint" "WMS_components:TP4056-18650_v2" (at 36.83 25.4 0)
       (effects (font (size 1.27 1.27)) hide)
     )
@@
       (effects (font (size 1.27 1.27)) hide)
     )
+    (pin "1")
+    (pin "2")
+    (pin "3")
     (pin "4")
-    (pin "1")
     (pin "5")
     (pin "6")
-    (pin "3")
-    (pin "2")
     (instances
       (project "WMS"
@@
       (effects (font (size 1.27 1.27)) hide)
     )
-    (property "Footprint" "WMS_components:MT3608_module" (at 87.63 24.13 0)
+    (property "Footprint" "WMS_components:MT3608_module_v2" (at 87.63 24.13 0)
       (effects (font (size 1.27 1.27)) hide)
     )
@@
       (effects (font (size 1.27 1.27)) hide)
     )
+    (pin "1")
+    (pin "2")
     (pin "3")
     (pin "4")
-    (pin "2")
-    (pin "1")
     (instances
       (project "WMS"
