File: PCB/WMS/WMS/WMS.kicad_pcb (KiCad board)
At the start: 2 copper layers, 173 x 163.6 mm, 32 parts, among them J1 Conn_01x40_Socket, J2 Conn_01x40_Socket, J3 Conn_01x03_Socket, J4 Conn_02x06_Odd_Even, J5 Conn_02x06_Odd_Even, SW1 SW_Push_Open, SW2 SW_Push_DPDT, SW3 SW_Push_Open, SW4 SW_SPDT

Commit message: +Update PCB (v.1)
membuat PCB versi 1
Parts:
- added U7: ~, WMS_components:YR903_RFID_Scanner_FPC, F.Cu at (119.8, 103.9)
- Brd1: footprint WMS_components:128x64OLED -> WMS_components:128x64OLED_v2
- U1: footprint WMS_components:YX850 -> WMS_components:YX850_v2
- U2: footprint WMS_components:MT3608_module -> WMS_components:MT3608_module_v2
- U3: footprint WMS_components:TP4056-18650 -> WMS_components:TP4056-18650_v2
- U5: footprint WMS_components:GM67_Barcode_Scanner -> WMS_components:Quad_SPI_flash_microSD_v2; moved to F.Cu
- U6: footprint WMS_components:CY8CPROTO-062-4343W -> WMS_components:CY8CPROTO-062-4343W_v2
- moved U5 133.9 mm to (44.2, 96.3), turned to 0 degrees
- moved H1 58.0 mm to (42.7, 87.9)
- moved H3 51.3 mm to (46.5, 170.9)
- moved H4 21.1 mm to (43.2, 145.3)
- moved U1 16.4 mm to (17.5, 47.8)
- moved Brd1 13.5 mm to (186.8, 72.6)
- moved H2 11.9 mm to (42.4, 66.3)
- moved J1 10.4 mm to (78.5, 65.4)
- moved J2 9.91 mm to (47.8, 65.6)
Connections:
- U5 pad 1: /PCB1 : Subsistem Data Processing, Gateway, Power/POWER_RFID -> GND
- U5 pad 2: GND -> P13_5
- U5 pad 3: P12_0 -> P13_4
- U5 pad 4: P12_1 -> P13_0
Other:
- board size 173 x 163.6 mm -> 180 x 146 mm
